File: hardware/v2/Car.sch (EAGLE design)
At the start: 72 parts

Commit message: More updates to schematic and layout. Checkpointing.
Parts:
- removed C11, C9, PSB2: 1u, rcl:C-USC0805
- removed U$2: MCP6L2-X_SN, microchip2:MCP6L2-X_SN
- added C6, C7, C8: 1u, rcl:C-USC1206
- added M1_LPF1: MCP6L2-X_SN, microchip2:MCP6L2-X_SN
- added M2_CA, M2_CB: 100nF, rcl:C-USC0805
- added M2_R1A, M2_R1B: 105k, rcl:R-US_R0805
- added M2_R2A, M2_R2B: 200k, rcl:R-US_R0805
- added M2_RA, M2_RB: 22k, rcl:R-US_R0805
- M1_CA, M1_CB: value 1n -> 100nF
- M1_R1A, M1_R1B: value 2k -> 105k
- M1_R2A, M1_R2B: value 2k -> 200k
- M1_RA, M1_RB: value 2k -> 22k
- RL1, RL2: value 1k -> 2k
- RN1: value 10k -> 22k
- renumbered CA to M1_CA, CB to M1_CB, RA to M1_RA, RB to M1_RB, RFA to M1_R1A, RFB to M1_R1B, RGA to M1_R2A, RGB to M1_R2B, U$1 to M1_LPF
Connections:
- new net N$12: M1_LPF1.VINA+, M2_CA.1, M2_RA.1
- new net N$19: M1_LPF1.VINA-, M2_R1A.2
- new net N$23: M1_LPF1.VINB-, M2_R1B.2
- new net N$24: M1_LPF1.VINB+, M2_CB.1, M2_RB.1
- net 12V: now also C6.1; no longer PSB2.1
- net 3V3: now also C7.1; no longer C9.1
- net 5V: now also C8.1, M1_LPF1.VDD; no longer C11.1
- net AGND: now also M1_LPF1.VSS, M2_CA.2, M2_CB.2, M2_R2A.2, M2_R2B.2
- net GND: now also C6.2, C7.2, C8.2; no longer C11.2, C9.2, PSB2.2
- net M2_PWM1: now also M2_RA.2
- net M2_PWM2: now also M2_RB.2
- net M2_V1: now also M1_LPF1.VOUTA, M2_R1A.1, M2_R2A.1
- net M2_V2: now also M1_LPF1.VOUTB, M2_R1B.1, M2_R2B.1

Commit message: Started routing pcb for reals.
Parts:
- removed 3V3, 5V: 317EMP, linear:317EMP
- added U$1, U$2: LM317, misc:LM317
- M1_CA, M1_CB, M2_CA, M2_CB: value 100nF -> 100n
Connections:
- net 12V: now also U$1.VI, U$2.VI; no longer 3V3.VI, 5V.VI
- net 3V3: now also U$2.VO; no longer 3V3.VO
- net 5V: now also U$1.VO; no longer 5V.VO
- net GND: now also J1.2
- net N$20: now also U$2.ADJ; no longer 3V3.ADJ
- net N$27: now also U$1.ADJ; no longer 5V.ADJ

Commit message: Finished routing power signals.
Parts:
- AIO: value M10LOCK -> (none); device SparkFun-Connectors:M10LOCK -> SparkFun-Connectors:M11LOCK
- renumbered C6 to PSB2, H1 to MD1, H2 to MD2, M1_LPF1 to M2_LPF, U$1 to 5V, U$2 to 3V3
Connections:
- net 3V3: now also AIO.10; no longer AIO.1
- net 5V: now also AIO.11
- net A0: now also AIO.8; no longer AIO.3
- net A1: now also AIO.7; no longer AIO.4
- net A2: now also AIO.6; no longer AIO.5
- net A3: now also AIO.5; no longer AIO.6
- net A4: now also AIO.4; no longer AIO.7
- net A5: now also AIO.3; no longer AIO.8
- net A6: now also AIO.2; no longer AIO.9
- net A7: now also AIO.1; no longer AIO.10
- net DGND: now also AIO.9; no longer AIO.2

Commit message: Finalized(-ish) routing for V2
Parts:
- added R1: 1k, rcl:R-US_R0805
- added T1: (no value), transistor:BC817-16-NPN-SOT23-BEC
- renumbered M.ARMS to HIPS, MD1 to LEGS1, MD2 to LEGS2
Connections:
- new net N$26: AIO.2, T1.C
- new net N$28: R1.1, T1.B
- net A6: now also R1.2; no longer AIO.2
- net DGND: now also T1.E
