File: hardware/v3/Car.sch (EAGLE design)
At the start: 75 parts, among them IC1 PIC24FJ64GB204, IC2 LD117AS50TR, IC3 LD117AS33TR

Commit message: Finished routing power for motor driver 1.
Parts:
- 11RS, 21RS: value 1 -> 0.5
Changed lines of the file:
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@@
 <part name="MD1" library="microchip" deviceset="MTS62C19A" device=""/>
 <part name="MD2" library="microchip" deviceset="MTS62C19A" device=""/>
-<part name="11RS" library="resistor" deviceset="R-US_" device="R1210" value="1"/>
+<part name="11RS" library="resistor" deviceset="R-US_" device="R1210" value="0.5"/>
 <part name="12RS" library="resistor" deviceset="R-US_" device="R1210" value="1"/>
 <part name="11RC" library="rcl" deviceset="R-US_" device="R0805" value="2k"/>
@@
 <part name="22CC" library="rcl" deviceset="C-US" device="C0805" value="1n"/>
 <part name="R22" library="rcl" deviceset="R-US_" device="R0805" value="2k"/>
-<part name="21RS" library="resistor" deviceset="R-US_" device="R1210" value="1"/>
+<part name="21RS" library="resistor" deviceset="R-US_" device="R1210" value="0.5"/>
 <part name="22RS" library="resistor" deviceset="R-US_" device="R1210" value="1"/>
 <part name="C13" library="rcl" deviceset="C-US" device="C0805" value="100n"/>

Commit message: Finished routing power lines and other significant signals.
Parts:
- removed JP1: (no value), SparkFun-Connectors:M04LOCK
- added C31, C32, C33, C34: 1n, rcl:C-USC0805
- added PIO: (no value), SparkFun-Connectors:M05LOCK
- added R31, R32, R33, R34: 2k, rcl:R-US_R0805
- 12RS, 22RS: value 1 -> 0.5
- R23, R25: value 1k -> 10k
- T1, T2: value (none) -> 2N3904
- renumbered IC2 to VR1, IC3 to VR2, JP6 to PWR_IN, JP7 to DIO1, JP8 to DIO2, JP9 to AIO
Connections:
- new net M1_VREF1: C31.1, MD1.VREF1, R31.2
- new net M1_VREF2: C32.1, MD1.VREF2, R32.2
- new net M2_VREF1: C33.1, MD2.VREF1, R33.2
- new net M2_VREF2: C34.1, MD2.VREF2, R34.2
- net +3V3: now also PIO.1
- net +5V: now also PIO.2; no longer JP1.1, R24.2, R26.2
- net A4_PO: now also PIO.3, R24.2; no longer JP1.2, T1.E
- net A5_PO: now also PIO.4, R26.2; no longer JP1.3, T2.E
- net D10/M2_PWM2: now also R34.1; no longer MD2.VREF2
- net D5/M1_PWM1: now also R31.1; no longer MD1.VREF1
- net D6/M1_PWM2: now also R32.1; no longer MD1.VREF2
- net D9/M2_PWM1: now also R33.1; no longer MD2.VREF1
- net GND: now also C31.2, C32.2, C33.2, C34.2, PIO.5, T1.E, T2.E; no longer JP1.4
Other:
- note added: "*see datasheet for dual powering options"
- note removed: "*see datasheet for dual power circuit"
- moved on the sheet: C11, C13, C23, C24, C25, C26, C41, D1, F1, F2, J1, R23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
